File: protomono_pcb/protomono_pcb.kicad_sch (KiCad schematic)
At the start: 93 parts, among them SW1 SW_PUSH, SW10 SW_PUSH, SW11 SW_PUSH, SW12 SW_PUSH, SW13 SW_PUSH, SW14 SW_PUSH, SW15 SW_PUSH, SW16 SW_PUSH, SW17 SW_PUSH, SW18 SW_PUSH, SW19 SW_PUSH, SW2 SW_PUSH, SW20 SW_PUSH, SW21 SW_PUSH, SW22 SW_PUSH, SW23 SW_PUSH, SW24 SW_PUSH, SW25 SW_PUSH, SW26 SW_PUSH, SW27 SW_PUSH, SW28 SW_PUSH, SW29 SW_PUSH, SW3 SW_PUSH, SW30 SW_PUSH, SW31 SW_PUSH, SW32 SW_PUSH, SW33 SW_PUSH, SW34 SW_PUSH, SW35 SW_PUSH, SW36 SW_PUSH, SW37 SW_PUSH, SW38 SW_PUSH, SW39 SW_PUSH, SW4 SW_PUSH, SW40 SW_PUSH, SW41 SW_PUSH, SW42 SW_PUSH, SW43 SW_PUSH, SW44 SW_PUSH, SW45 SW_PUSH, SW46 SW_PUSH, SW5 SW_PUSH, SW6 SW_PUSH, SW7 SW_PUSH, SW8 SW_PUSH, SW9 SW_PUSH, U1 ProMicro

Commit message: Start laying the PCB down
Other:
- note added: "index"
- note added: "middle"
- note added: "pinkie"
- note added: "ring"
- note added: "thumb"
- moved on the sheet: D1, D10, D11, D12, D13, D14, D15, D16, D17, D18, D19, D2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

Commit message: Use RP2040, remove one index key
Parts:
- removed D13, D24: BAT85, Diode_THT:D_DO-35_SOD27_P7.62mm_Horizontal, symbol Diode:BAT85
- removed SW13, SW24: SW_PUSH, KS33:keyswitch_gateron_low_profile_hotswap_1u, symbol KS33:SW_PUSH
- removed U1: ProMicro, KS33:ProMicro, symbol KS33:ProMicro
- added A1: RaspberryPi_Pico, Module:RaspberryPi_Pico_Common_Unspecified, symbol MCU_Module:RaspberryPi_Pico
- added D13: SK6812MINI, LED_SMD:LED_SK6812MINI_PLCC4_3.5x3.5mm_P1.75mm, symbol LED:SK6812MINI
- added R1, R2, R3, R4: R, symbol Device:R
Connections:
- net COL_13 is gone; now on net COL_11: SW38.1, SW42.1
- net COL_0: now also SW14.1, A1.11 (GPIO8)
- net COL_1: now also SW15.1, A1.12 (GPIO9); no longer SW14.1
- net COL_10: now also SW34.1, SW39.1, SW40.1, A1.29 (GPIO22); no longer SW28.1, SW32.1, SW36.1, SW46.1
- net COL_11: now also SW43.1, A1.31 (GPIO26_ADC0); no longer SW31.1, SW35.1, SW40.1
- net COL_2: now also SW16.1, SW45.1, A1.14 (GPIO10); no longer SW15.1
- net COL_3: now also SW17.1, SW20.1, A1.15 (GPIO11); no longer SW16.1, SW45.1
- net COL_4: now also SW18.1, SW21.1, A1.16 (GPIO12); no longer SW17.1, SW20.1
- net COL_5: now also SW19.1, SW22.1, A1.17 (GPIO13); no longer SW18.1, SW21.1
- net COL_6: now also SW23.1, SW26.1, SW27.1, SW37.1, A1.24 (GPIO18); no longer SW19.1, SW22.1
- net COL_7: now also SW25.1, SW29.1, SW30.1, SW41.1, A1.25 (GPIO19); no longer SW27.1, SW37.1
- net COL_8: now also SW28.1, SW32.1, SW33.1, SW44.1, A1.26 (GPIO20); no longer SW23.1, SW26.1, SW30.1, SW41.1
- net COL_9: now also SW31.1, SW35.1, SW36.1, SW46.1, A1.27 (GPIO21); no longer SW25.1, SW29.1, SW33.1, SW44.1
- net GND: now also A1.13 (GND), A1.18 (GND), A1.23 (GND), A1.28 (GND), A1.3 (GND), A1.33 (AGND), A1.38 (GND), A1.8 (GND)
- net ROW_0: now also A1.20 (GPIO15), R1.1; no longer D1.1 (K), D2.1 (K), D23.1 (K), D25.1 (K), D28.1 (K), D3.1 (K), D31.1 (K), D34.1 (K), D38.1 (K), D4.1 (K), D5.1 (K), D6.1 (K)
- net ROW_1: now also A1.19 (GPIO14), R2.1; no longer D10.1 (K), D11.1 (K), D12.1 (K), D26.1 (K), D29.1 (K), D32.1 (K), D35.1 (K), D39.1 (K), D42.1 (K), D7.1 (K), D8.1 (K), D9.1 (K)
- net ROW_2: now also A1.21 (GPIO16), R3.1; no longer D14.1 (K), D15.1 (K), D16.1 (K), D17.1 (K), D18.1 (K), D19.1 (K), D27.1 (K), D30.1 (K), D33.1 (K), D36.1 (K), D40.1 (K), D43.1 (K)
- net ROW_3: now also A1.22 (GPIO17), R4.1; no longer D20.1 (K), D21.1 (K), D22.1 (K), D37.1 (K), D41.1 (K), D44.1 (K), D45.1 (K), D46.1 (K)
- removed net COL_12: SW34.1, SW39.1, SW43.1
- new net: D1.1 (K), D2.1 (K), D23.1 (K), D25.1 (K), D28.1 (K), D3.1 (K), D31.1 (K), D34.1 (K), D38.1 (K), D4.1 (K), D5.1 (K), D6.1 (K), R1.2
- new net: D14.1 (K), D15.1 (K), D16.1 (K), D17.1 (K), D18.1 (K), D19.1 (K), D27.1 (K), D30.1 (K), D33.1 (K), D36.1 (K), D40.1 (K), D43.1 (K), R3.2
- new net: D10.1 (K), D11.1 (K), D12.1 (K), D26.1 (K), D29.1 (K), D32.1 (K), D35.1 (K), D39.1 (K), D42.1 (K), D7.1 (K), D8.1 (K), D9.1 (K), R2.2
- new net: D20.1 (K), D21.1 (K), D22.1 (K), D37.1 (K), D41.1 (K), D44.1 (K), D45.1 (K), D46.1 (K), R4.2
- no-connect marks 3 -> 16
