File: pcb/protomonopcb.kicad_pcb (KiCad board)
At the start: 2 copper layers, 149 parts

Commit message: Just another periodic push
Parts:
- removed LED1, LED10, LED11, LED12, LED13, LED14, LED15, LED16, LED17, LED18, LED19, LED2, LED20, LED21, LED22, LED23, LED24, LED26, LED27, LED28, LED29, LED3, LED30, LED31, LED32, LED33, LED34, LED35, LED37, LED38, LED39, LED4, LED40, LED41, LED42, LED43, LED44, LED45, LED46, LED47, LED48, LED49, LED5, LED50, LED6, LED7, LED8, LED9: SK6812MINI-E, LED_SMD:LED_SK6812MINI_PLCC4_3.5x3.5mm_P1.75mm
- added D25: LED, LED_THT:LED_D3.0mm, F.Cu at (195.2, 180.7)
- added D36: LED, LED_THT:LED_D3.0mm, F.Cu at (200.7, 180.7)
- added D51: LED, LED_THT:LED_D3.0mm, F.Cu at (206.3, 180.7)
- added D52: LED, LED_THT:LED_D3.0mm, F.Cu at (211.6, 180.7)
- added R5: 1k, Resistor_THT:R_Axial_DIN0204_L3.6mm_D1.6mm_P7.62mm_Horizontal, F.Cu at (195.2, 167.4)
- added R6: 1k, Resistor_THT:R_Axial_DIN0204_L3.6mm_D1.6mm_P7.62mm_Horizontal, F.Cu at (200.7, 167.4)
- added R7: 1k, Resistor_THT:R_Axial_DIN0204_L3.6mm_D1.6mm_P7.62mm_Horizontal, F.Cu at (206.3, 167.4)
- added R8: 1k, Resistor_THT:R_Axial_DIN0204_L3.6mm_D1.6mm_P7.62mm_Horizontal, F.Cu at (211.6, 167.4)
- A1: footprint Module:RaspberryPi_Pico_Common_Unspecified -> pico_without_keepout_area:RaspberryPi_Pico_Common_Unspecified
- CH1, CH13, CH14, CH15, CH16, CH17, CH18, CH2, CH26, CH27, CH28, CH29, CH3, CH30, CH37, CH38, CH39, CH4, CH40, CH41, CH42, CH49, CH5, CH6: footprint PCM_marbastlib-xp-gateron_lp:SW_KS33_HS_KS-2P02B01-02_HS_1u -> packed_switches_library:SW_KS33_HS_1u_18.5mm; moved to B.Cu
- CH10, CH11, CH12, CH19, CH20, CH21, CH22, CH23, CH24, CH31, CH32, CH33, CH34, CH35, CH43, CH44, CH45, CH46, CH47, CH48, CH50, CH7, CH8, CH9: footprint PCM_marbastlib-xp-gateron_lp:SW_KS33_HS_KS-2P02B01-02_HS_1u -> packed_switches_library:SW_KS33_HS_1u_18.5mm
- moved D38 263.9 mm to (181.3, 59.4), turned to 90 degrees
- moved D29 242.5 mm to (166.1, 59.4), turned to 90 degrees
- moved D37 241.8 mm to (145.7, 59.4), turned to 90 degrees
- moved D30 241.1 mm to (155.9, 59.4), turned to 90 degrees
- moved D42 235.7 mm to (171.1, 59.4), turned to 90 degrees
- moved D41 233.6 mm to (173.7, 59.4), turned to 90 degrees
- moved D28 233.6 mm to (153.4, 59.4), turned to 90 degrees
- moved D40 231.5 mm to (176.2, 59.4), turned to 90 degrees
- moved D39 229.5 mm to (178.8, 59.4), turned to 90 degrees
- moved D6 228.4 mm to (163.5, 59.4), turned to 90 degrees
- moved D27 226.1 mm to (143.2, 59.4), turned to 90 degrees
- moved D5 223.4 mm to (158.4, 59.4), turned to 90 degrees
- moved D11 222.4 mm to (280.9, 59.4), turned to 90 degrees
- moved D13 221.0 mm to (128.0, 59.4), turned to 90 degrees
- moved D26 220.8 mm to (138.1, 59.4), turned to 90 degrees
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Connections:
- A1 pad 1: LED_in -> LED_0
- A1 pad 12: Net-(A1-GPIO9) -> c0
- A1 pad 14: c0 -> c1
- A1 pad 15: c1 -> c2
- A1 pad 16: c2 -> c3
- A1 pad 17: c3 -> c4
- A1 pad 19: c4 -> c5
- A1 pad 2: unconnected-(A1-GPIO1-Pad2)_1 -> LED_1
- A1 pad 20: c5 -> ci
- A1 pad 21: c6 -> cii
- A1 pad 22: c7 -> c6
- A1 pad 24: c8 -> c7
- A1 pad 25: c9 -> c8
- A1 pad 26: c10 -> c9
- A1 pad 27: c11 -> c10
- A1 pad 29: unconnected-(A1-GPIO22-Pad29) -> c11
- A1 pad 4: unconnected-(A1-GPIO2-Pad4)_1 -> LED_2
- A1 pad 5: unconnected-(A1-GPIO3-Pad5)_1 -> LED_3
- A1 pad 7: unconnected-(A1-GPIO5-Pad7)_1 -> Net-(A1-GPIO5)
- CH29 pad 1: c4 -> c5
- CH30 pad 1: c5 -> c4
- CH37 pad 1: c1 -> c2
- CH38 pad 1: c2 -> c4
- CH39 pad 1: c3 -> c5
- CH40 pad 1: c4 -> ci
- CH41 pad 1: c5 -> ci
- CH42 pad 1: c8 -> ci
- CH43 pad 1: c9 -> cii
- CH44 pad 1: c10 -> c9
- CH45 pad 1: c7 -> cii
- CH47 pad 1: c0 -> c7
- CH48 pad 1: c11 -> cii
- CH49 pad 1: c0 -> c1
- CH50 pad 1: c11 -> c10
- D1 pad 2: r2 -> r0
- D10 pad 2: r3 -> r0
- D11 pad 2: r3 -> r1
- D12 pad 2: r2 -> r0
- D15 pad 2: r2 -> r1
- D16 pad 2: r2 -> r1
- D17 pad 2: r2 -> r1
- D18 pad 2: r2 -> r1
- D19 pad 2: r2 -> r1
- D2 pad 2: r3 -> r1
- D20 pad 2: r2 -> r1
- D21 pad 2: r2 -> r1
- D22 pad 2: r2 -> r1
- D26 pad 2: r1 -> r3
- D27 pad 2: r1 -> r2
- D28 pad 2: r1 -> r2
- D29 pad 2: r1 -> r2
- D3 pad 2: r3 -> r0
- D30 pad 2: r1 -> r2
- D31 pad 2: r1 -> r2
- D32 pad 2: r1 -> r2
- D33 pad 2: r1 -> r2
- D34 pad 2: r1 -> r2
- D35 pad 2: r1 -> r3
- D37 pad 2: r0 -> r3
- D38 pad 2: r0 -> r3
- D39 pad 2: r0 -> r3
- D4 pad 2: r3 -> r0
- D40 pad 2: r0 -> r3
- D41 pad 2: r0 -> r2
- D42 pad 2: r0 -> r1
- D43 pad 2: r0 -> r2
- D44 pad 2: r0 -> r3
- D45 pad 2: r0 -> r3
- D46 pad 2: r0 -> r3
- D47 pad 2: r0 -> r3
- D48 pad 2: r0 -> r1
- D49 pad 2: r3 -> r0
- D5 pad 2: r3 -> r0
- D50 pad 2: r3 -> r0
- D6 pad 2: r3 -> r0
- D7 pad 2: r3 -> r0
- D8 pad 2: r3 -> r0
- D9 pad 2: r3 -> r0
- R1 pad 1: Net-(A1-GPIO6) -> Net-(A1-GPIO5)
- R2 pad 1: Net-(A1-GPIO7) -> Net-(A1-GPIO6)
- R3 pad 1: Net-(A1-GPIO8) -> Net-(A1-GPIO7)
- R4 pad 1: Net-(A1-GPIO9) -> Net-(A1-GPIO8)
Routing:
- net r1: track 0.00 -> 298.0 mm
- net r0: track 0.00 -> 296.3 mm
- net r2: track 0.00 -> 269.1 mm
- net r3: track 0.00 -> 255.4 mm
- net c1: track 0.00 -> 204.7 mm
- net c0: track 0.00 -> 196.7 mm
- net c10: track 0.00 -> 192.3 mm
- net Net-(D47-K): track 0.00 -> 190.2 mm
- net Net-(D38-K): track 0.00 -> 188.5 mm
- net c11: track 0.00 -> 185.3 mm
- net Net-(D39-K): track 0.00 -> 168.5 mm
- net c2: track 0.00 -> 162.0 mm
- net Net-(D40-K): track 0.00 -> 147.7 mm
- net c9: track 0.00 -> 145.3 mm
- net c4: track 0.00 -> 121.5 mm
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Other:
- board outline added: 297.9 x 140.6 mm

Commit message: Bottom PCB completed
Parts:
- removed D25, D36, D51, D52: LED, LED_THT:LED_D3.0mm
- removed R5, R6, R7, R8: 1k, Resistor_THT:R_Axial_DIN0204_L3.6mm_D1.6mm_P7.62mm_Horizontal
- added H1: MountingHole, MountingHole:MountingHole_3.2mm_M3_Pad_Via, F.Cu at (222.0, 140.6)
- added H10: MountingHole, MountingHole:MountingHole_3.2mm_M3_Pad_Via, F.Cu at (349.6, 68.5)
- added H11: MountingHole, MountingHole:MountingHole_3.2mm_M3_Pad_Via, F.Cu at (83.9, 127.1)
- added H2: MountingHole, MountingHole:MountingHole_3.2mm_M3_Pad_Via, F.Cu at (333.0, 155.4)
- added H3: MountingHole, MountingHole:MountingHole_3.2mm_M3_Pad_Via, F.Cu at (92.5, 68.5)
- added H4: MountingHole, MountingHole:MountingHole_3.2mm_M3_Pad_Via, F.Cu at (203.4, 55.4)
- added H5: MountingHole, MountingHole:MountingHole_3.2mm_M3_Pad_Via, F.Cu at (199.8, 193.1)
- added H6: MountingHole, MountingHole:MountingHole_3.2mm_M3_Pad_Via, F.Cu at (111.0, 155.4)
- added H7: MountingHole, MountingHole:MountingHole_3.2mm_M3_Pad_Via, F.Cu at (359.9, 126.9)
- added H8: MountingHole, MountingHole:MountingHole_3.2mm_M3_Pad_Via, F.Cu at (240.5, 55.5)
- added H9: MountingHole, MountingHole:MountingHole_3.2mm_M3_Pad_Via, F.Cu at (244.8, 193.1)
- moved CH32 22.3 mm to (288.0, 136.9)
- moved CH42 22.3 mm to (200.2, 134.5)
- moved D31 22.3 mm to (265.1, 73.6)
- moved CH10 22.3 mm to (311.4, 84.8)
- moved CH20 22.3 mm to (278.8, 120.8)
- moved CH21 22.3 mm to (290.2, 103.6)
- moved CH22 22.3 mm to (316.2, 102.7)
- moved CH31 22.3 mm to (273.9, 149.3)
- moved CH33 22.3 mm to (299.4, 119.6)
- moved CH41 22.3 mm to (190.9, 150.5)
- moved CH46 22.3 mm to (279.1, 167.6)
- moved CH9 22.3 mm to (280.9, 87.5)
- moved D11 22.3 mm to (298.1, 73.6)
- moved D17 22.3 mm to (178.2, 73.6)
- moved D23 22.3 mm to (290.5, 73.6)
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Routing:
- net GND: track 0.00 -> 104.1 mm
- net Net-(D43-K): track 100.3 -> 105.5 mm
- net Net-(D11-K): track 72.2 -> 75.8 mm
- net Net-(D52-A): track 3.15 -> 0.00 mm
- net Net-(D36-A): track 3.15 -> 0.00 mm
- net Net-(D25-A): track 3.15 -> 0.00 mm
- net Net-(D51-A): track 3.13 -> 0.00 mm
- net Net-(D32-K): track 85.0 -> 82.0 mm
- net c10: track 192.3 -> 189.5 mm
- net Net-(D33-K): track 66.0 -> 63.6 mm
- net c11: track 185.3 -> 183.1 mm
- net Net-(D22-K): track 65.8 -> 63.8 mm
- net Net-(D34-K): track 84.1 -> 82.6 mm
- net c0: track 196.7 -> 195.4 mm
- net Net-(D24-K): track 109.2 -> 110.2 mm
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Other:
- board size 297.9 x 140.6 mm -> 296 x 151.7 mm
